Commit message: update atlas.urdf

File: urdf/atlas_description/urdf/atlas.urdf (robot description, URDF)
Before this commit: robot drc_skeleton, 28 links, 28 joints
Links:
- removed link l_farm
- removed link r_farm
- added link center_bottom_led_frame, mass 1e-5
- added link center_top_led_frame, mass 1e-5
- added link head, mass 1.41984; collision box size=0.0468 0.12 0.1184; collision box size=0.1311 0.12 0.0591
- added link head_hokuyo_frame, mass 1e-5
- added link head_imu_link, mass 1e-5; visual box size=0.01 0.01 0.01
- added link hokuyo_link, mass 0.057654; collision box size=0.08 0.06 0.04238; collision cylinder length=0.047 radius=0.024425
- added link imu_link, mass 0.1; visual box size=0.01 0.01 0.01
- added link l_lfarm, mass 1.6; collision cylinder length=0.015 radius=0.045; collision cylinder length=0.015 radius=0.052
- added link l_situational_awareness_camera_link, mass 0.1; visual box size=0.01 0.01 0.01
- added link l_situational_awareness_camera_optical_frame
- added link l_ufarm, mass 2.4798; collision box size=0.08 0.09 0.11; collision cylinder length=0.1 radius=0.053
- added link left_camera_frame, mass 1e-5
- added link left_camera_optical_frame
- added link left_led_frame, mass 1e-5
- added link r_lfarm, mass 1.6; collision cylinder length=0.015 radius=0.045; collision cylinder length=0.015 radius=0.052
- added link r_situational_awareness_camera_link, mass 0.1; visual box size=0.01 0.01 0.01
- added link r_situational_awareness_camera_optical_frame
- added link r_ufarm, mass 2.4798; collision box size=0.08 0.09 0.11; collision cylinder length=0.1 radius=0.053
- added link right_camera_frame, mass 1e-5
- added link right_camera_optical_frame
- added link right_led_frame, mass 1e-5
- link l_clav: mass 2.369 -> 4.466; geometry collision box size=0.1 0.07 0.072; collision cylinder length=0.1525 radius=0.0555
- link l_foot: mass 1.634 -> 2.410; geometry collision box size=0.1 0.08 0.02; collision box size=0.227 0.133887 0.05
- link l_hand: mass 2.263 -> 1.7839; geometry 
- link l_larm: mass 2.148 -> 3.248; geometry collision box size=0.025 0.06 0.06; collision box size=0.025 0.155 0.07
- link l_lglut: mass 0.69 -> 0.898; geometry collision box size=0.0975 0.069 0.103; collision box size=0.125 0.05 0.08
- link l_lleg: mass 4.367 -> 4.515; geometry collision cylinder length=0.40 radius=0.07; visual mesh filename=package://atlas_description/meshes_unplugged/l_lleg.dae
- link l_scap: mass 2.707 -> 3.899; geometry collision box size=0.02 0.029 0.018; collision box size=0.028 0.090 0.05
- link l_talus: mass 0.1 -> 0.125; geometry collision cylinder length=0.010059 radius=0.010348; collision cylinder length=0.029542 radius=0.010181
- link l_uarm: mass 1.881 -> 4.386; geometry collision box size=0.05 0.07 0.15; collision cylinder length=0.11 radius=0.065
- link l_uglut: mass 0.5166 -> 1.959; geometry collision box size=0.05 0.1 0.1; collision cylinder length=0.080842 radius=0.019841
- link l_uleg: mass 7.34 -> 8.204; geometry collision box size=0.07 0.038 0.14; collision box size=0.07 0.038 0.15
- link ltorso: mass 1.92 -> 2.270; geometry visual mesh filename=package://atlas_description/meshes_unplugged/ltorso.dae
- link mtorso: mass 0.55 -> 0.799; geometry collision cylinder length=0.15 radius=0.02; visual mesh filename=package://atlas_description/meshes_unplugged/mtorso.dae
- link pelvis: mass 14.2529 -> 9.509; geometry collision box size=0.1 0.15 0.2; collision cylinder length=0.05 radius=0.16
- link r_clav: mass 2.369 -> 4.466; geometry collision box size=0.1 0.07 0.072; collision cylinder length=0.1525 radius=0.0555
- link r_foot: mass 1.634 -> 2.41; geometry collision box size=0.1 0.08 0.02; collision box size=0.227 0.133887 0.05
- link r_hand: mass 2.263 -> 1.7839; geometry 
- link r_larm: mass 2.148 -> 3.248; geometry collision box size=0.025 0.06 0.06; collision box size=0.025 0.155 0.07
- link r_lglut: mass 0.69 -> 0.898; geometry collision box size=0.0975 0.069 0.103; collision box size=0.125 0.05 0.08
- link r_lleg: mass 4.367 -> 4.515; geometry collision cylinder length=0.40 radius=0.07; visual mesh filename=package://atlas_description/meshes_unplugged/r_lleg.dae
- link r_scap: mass 2.707 -> 3.899; geometry collision box size=0.02 0.029 0.018; collision box size=0.028 0.090 0.05
- link r_talus: mass 0.1 -> 0.125; geometry collision cylinder length=0.010059 radius=0.010348; collision cylinder length=0.029542 radius=0.010181
- link r_uarm: mass 1.881 -> 4.386; geometry collision box size=0.05 0.07 0.15; collision cylinder length=0.11 radius=0.065
- link r_uglut: mass 0.5166 -> 1.959; geometry collision box size=0.05 0.1 0.1; collision cylinder length=0.080842 radius=0.019841
- link r_uleg: mass 7.34 -> 8.204; geometry collision box size=0.07 0.038 0.14; collision box size=0.07 0.038 0.15
- link utorso: mass 18.484 -> 84.409; geometry collision box size=0.13 0.50 0.10; collision box size=0.2 0.18 0.10
Joints:
- removed joint back_lbz
- removed joint back_mby
- removed joint back_ubx
- removed joint l_arm_mwx
- removed joint l_arm_usy
- removed joint l_arm_uwy
- removed joint l_leg_lax
- removed joint l_leg_lhy
- removed joint l_leg_mhx
- removed joint l_leg_uay
- removed joint l_leg_uhz
- removed joint neck_ay
- removed joint r_arm_mwx
- removed joint r_arm_usy
- removed joint r_arm_uwy
- removed joint r_leg_lax
- removed joint r_leg_lhy
- removed joint r_leg_mhx
- removed joint r_leg_uay
- removed joint r_leg_uhz
- added joint back_bkx: type revolute, parent mtorso, child utorso, origin xyz=0 0 0.05 rpy=0 0 0, axis 1 0 0, limit lower=-0.523599 upper=0.523599 effort=300 velocity=12
- added joint back_bky: type revolute, parent ltorso, child mtorso, origin xyz=0 0 0.162 rpy=0 0 0, axis 0 1 0, limit lower=-0.219388 upper=0.538783 effort=445 velocity=9
- added joint back_bkz: type revolute, parent pelvis, child ltorso, origin xyz=-0.0125 0 0 rpy=0 0 0, axis 0 0 1, limit lower=-0.663225 upper=0.663225 effort=106 velocity=12
- added joint center_bottom_led_frame_joint: type fixed, parent head, child center_bottom_led_frame, origin xyz=0.01125 0.0 -0.0155
- added joint center_top_led_frame_joint: type fixed, parent head, child center_top_led_frame, origin xyz=0.01125 0.0 0.0105
- added joint head_hokuyo_joint: type fixed, parent hokuyo_link, child head_hokuyo_frame, origin xyz=0.03 0 0.015 rpy=0 0 0, axis 0 1 0
- added joint head_imu_joint: type fixed, parent head, child head_imu_link, origin xyz=-0.0475 0.035 0.0 rpy=0 0 0
- added joint hokuyo_joint: type continuous, parent head, child hokuyo_link, origin xyz=-0.0446 0 0.0880 rpy=0 0 0, axis 1 0 0
- added joint imu_joint: type fixed, parent pelvis, child imu_link, origin xyz=0 0 0 rpy=0 0 0
- added joint l_arm_shz: type revolute, parent utorso, child l_clav, origin xyz=0.1406 0.2256 0.4776 rpy=0 0 0, axis 0 0 1, limit lower=-1.5708 upper=0.785398 effort=87 velocity=12
- added joint l_arm_wrx: type revolute, parent l_ufarm, child l_lfarm, origin xyz=0 0 0 rpy=0 0 0, axis 1 0 0, limit lower=-1.7628 upper=1.7628 effort=25 velocity=10
- added joint l_arm_wry: type revolute, parent l_larm, child l_ufarm, origin xyz=0 0.29955 -0.00921 rpy=0 0 0, axis 0 1 0, limit lower=-3.011 upper=3.011 effort=25 velocity=10
- added joint l_arm_wry2: type revolute, parent l_lfarm, child l_hand, origin xyz=0 0 0 rpy=0 0 0, axis 0 1 0, limit lower=-2.9671 upper=2.9671 effort=25 velocity=10
- added joint l_leg_akx: type revolute, parent l_talus, child l_foot, origin xyz=0 0 0 rpy=0 0 0, axis 1 0 0, limit lower=-0.8 upper=0.8 effort=360 velocity=12
- added joint l_leg_aky: type revolute, parent l_lleg, child l_talus, origin xyz=0 0 -0.422 rpy=0 0 0, axis 0 1 0, limit lower=-1 upper=0.7 effort=740 velocity=12
- added joint l_leg_hpx: type revolute, parent l_uglut, child l_lglut, origin xyz=0 0 0 rpy=0 0 0, axis 1 0 0, limit lower=-0.523599 upper=0.523599 effort=530 velocity=12
- added joint l_leg_hpy: type revolute, parent l_lglut, child l_uleg, origin xyz=0.05 0.0225 -0.066 rpy=0 0 0, axis 0 1 0, limit lower=-1.61234 upper=0.65764 effort=840 velocity=12
- added joint l_leg_hpz: type revolute, parent pelvis, child l_uglut, origin xyz=0 0.089 0 rpy=0 0 0, axis 0 0 1, limit lower=-0.174358 upper=0.786794 effort=275 velocity=12
- added joint l_situational_awareness_camera_joint: type fixed, parent utorso, child l_situational_awareness_camera_link, origin xyz=0.155 0.121 0.785 rpy=0 0 1.309
- added joint l_situational_awareness_camera_optical_frame_joint: type fixed, parent l_situational_awareness_camera_link, child l_situational_awareness_camera_optical_frame, origin xyz=0 0 0 rpy=-1.5708 0.0 -1.5708
- added joint left_camera_frame_joint: type fixed, parent head, child left_camera_frame, origin xyz=0.0 0.035 -0.002
- added joint left_camera_optical_frame_joint: type fixed, parent left_camera_frame, child left_camera_optical_frame, origin xyz=0 0 0 rpy=-1.5708 0.0 -1.5708
- added joint left_led_frame_joint: type fixed, parent head, child left_led_frame, origin xyz=-0.01443 0.07452 0.050346 rpy=0 -0.15 0.53
- added joint neck_ry: type revolute, parent utorso, child head, origin xyz=0.2546 0 0.6215 rpy=0 0 0, axis 0 1 0, limit lower=-0.602139 upper=1.14319 effort=25 velocity=6.28
- added joint r_arm_shz: type revolute, parent utorso, child r_clav, origin xyz=0.1406 -0.2256 0.4776 rpy=0 0 0, axis 0 0 1, limit lower=-0.785398 upper=1.5708 effort=87 velocity=12
- added joint r_arm_wrx: type revolute, parent r_ufarm, child r_lfarm, origin xyz=0 0 0 rpy=0 0 0, axis 1 0 0, limit lower=-1.7628 upper=1.7628 effort=25 velocity=10
- added joint r_arm_wry: type revolute, parent r_larm, child r_ufarm, origin xyz=0 -0.29955 -0.00921 rpy=0 0 0, axis 0 1 0, limit lower=-3.011 upper=3.011 effort=25 velocity=10
- added joint r_arm_wry2: type revolute, parent r_lfarm, child r_hand, origin xyz=0 0 0 rpy=0 0 0, axis 0 1 0, limit lower=-2.9671 upper=2.9671 effort=25 velocity=10
- added joint r_leg_akx: type revolute, parent r_talus, child r_foot, origin xyz=0 0 0 rpy=0 0 0, axis 1 0 0, limit lower=-0.8 upper=0.8 effort=360 velocity=12
- added joint r_leg_aky: type revolute, parent r_lleg, child r_talus, origin xyz=0 0 -0.422 rpy=0 0 0, axis 0 1 0, limit lower=-1 upper=0.7 effort=740 velocity=12
- added joint r_leg_hpx: type revolute, parent r_uglut, child r_lglut, origin xyz=0 0 0 rpy=0 0 0, axis 1 0 0, limit lower=-0.523599 upper=0.523599 effort=530 velocity=12
- added joint r_leg_hpy: type revolute, parent r_lglut, child r_uleg, origin xyz=0.05 -0.0225 -0.066 rpy=0 0 0, axis 0 1 0, limit lower=-1.61234 upper=0.65764 effort=840 velocity=12
- added joint r_leg_hpz: type revolute, parent pelvis, child r_uglut, origin xyz=0 -0.089 0 rpy=0 0 0, axis 0 0 1, limit lower=-0.786794 upper=0.174358 effort=275 velocity=12
- added joint r_situational_awareness_camera_joint: type fixed, parent utorso, child r_situational_awareness_camera_link, origin xyz=0.155 -0.121 0.785 rpy=0 0 -1.309
- added joint r_situational_awareness_camera_optical_frame_joint: type fixed, parent r_situational_awareness_camera_link, child r_situational_awareness_camera_optical_frame, origin xyz=0 0 0 rpy=-1.5708 0.0 -1.5708
- added joint right_camera_frame_joint: type fixed, parent head, child right_camera_frame, origin xyz=0.0 -0.035 -0.002
- added joint right_camera_optical_frame_joint: type fixed, parent right_camera_frame, child right_camera_optical_frame, origin xyz=0 0 0 rpy=-1.5708 0.0 -1.5708
- added joint right_led_frame_joint: type fixed, parent head, child right_led_frame, origin xyz=-0.01443 -0.07452 0.050346 rpy=0 -0.15 -0.53
- joint l_arm_elx: limit lower=0 upper=2.35619 effort=114 velocity=12 -> lower=0 upper=2.35619 effort=112 velocity=12; origin xyz=0 0.121 0.013 rpy=0 -0 0 -> xyz=0 0.119 0.0092 rpy=0 0 0
- joint l_arm_ely: limit lower=0 upper=3.14159 effort=114 velocity=12 -> lower=0 upper=3.14159 effort=63 velocity=12; origin xyz=0 0.185 0 rpy=0 -0 0 -> xyz=0 0.187 -0.016 rpy=0 0 0
- joint l_arm_shx: limit lower=-1.39626 upper=1.74533 effort=170 velocity=12 -> lower=-1.5708 upper=1.5708 effort=99 velocity=12; origin xyz=0 0.075 0.036 rpy=0 -0 0 -> xyz=0 0.11 -0.245 rpy=0 0 0
- joint l_leg_kny: limit lower=0 upper=2.45 effort=220 velocity=12 -> lower=0 upper=2.35637 effort=890 velocity=12; origin xyz=-0.05 0 -0.374 rpy=0 -0 0 -> xyz=-0.05 0 -0.374 rpy=0 0 0
- joint r_arm_elx: limit lower=-2.35619 upper=0 effort=114 velocity=12 -> lower=-2.35619 upper=0 effort=112 velocity=12; origin xyz=0 -0.121 0.013 rpy=0 -0 0 -> xyz=0 -0.119 0.0092 rpy=0 0 0
- joint r_arm_ely: limit lower=0 upper=3.14159 effort=114 velocity=12 -> lower=0 upper=3.14159 effort=63 velocity=12; origin xyz=0 -0.185 0 rpy=0 -0 0 -> xyz=0 -0.187 -0.016 rpy=0 0 0
- joint r_arm_shx: limit lower=-1.74533 upper=1.39626 effort=170 velocity=12 -> lower=-1.5708 upper=1.5708 effort=99 velocity=12; origin xyz=0 -0.075 0.036 rpy=0 -0 0 -> xyz=0 -0.11 -0.245 rpy=0 0 0
- joint r_leg_kny: limit lower=0 upper=2.45 effort=220 velocity=12 -> lower=0 upper=2.35637 effort=890 velocity=12; origin xyz=-0.05 0 -0.374 rpy=0 -0 0 -> xyz=-0.05 0 -0.374 rpy=0 0 0
